File: arduino-uno-q-robotics.kicad_sch (KiCad schematic)
At the start: 19 parts, among them J1 Conn_02x30_Odd_Even, J2 Conn_02x30_Odd_Even, J3 Connector_FFC-FPC, J4 Connector_FFC-FPC, J5 Conn_02x30_Odd_Even, U1 LSM6DSO32, U2 TCA9803, U4 TCA9803

Commit message: Update to KiCAD 10
Parts:
- U3, U5, U6: value ~ -> (none)
